File: Hardware/APPS.kicad_pcb (KiCad board)
At the start: 2 copper layers, 100 x 63 mm, 88 parts, among them J1 Screw_Terminal_01x02, J2 Screw_Terminal_01x03, J3 Screw_Terminal_01x03, J4 Conn_01x06_Male, J5 Screw_Terminal_01x02, J6 Conn_01x06_Male, J7 Screw_Terminal_01x02, K1 FINDER-30.22, Q1 BSS138, SW1 SW_Push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

Commit message: Added Logos library, PCB FINISHED
Parts:
- added G***: LOGO, Logos:PUTM_LOGO_30mm, B.Cu at (155.6, 67.9)
- added G***: LOGO, Logos:SignatureBox37mm, B.Cu at (96.1, 99.9)
- added G***: LOGO, Logos:PUTM_LOGO_26mm, F.Cu at (158.9, 104.4)
Routing:
- net Net-(R21-Pad2): track 45.1 -> 44.2 mm, vias 0 -> 1
- net SW_GND: vias 11 -> 112
Other:
- board text added: "- Supply +"
- board text added: "3V3"
- board text added: "BT Conn"
- board text added: "CANH CANL"
- board text added: "GND"
- board text added: "GND1 POT1 SUP1"
- board text added: "GND2 POT2 SUP2"
- board text added: "IN safety OUT"
- board text added: "Jakub Jurczak"
- board text added: "NC"
- board text added: "NRST"
- board text added: "SWCLK"
- board text added: "SWDIO"
- board text added: "Szymon Sambor"
