File: Hardware/AnalogInputs.kicad_sch (KiCad schematic)
At the start: 12 parts, among them U7 MCP6001-OT, U8 MCP6001-OT

Commit message: Schematic cleanup
Parts:
- removed D11, D12: D_TVS_x2_AAC, Package_TO_SOT_SMD:SOT-23, symbol Device:D_TVS_x2_AAC
- added D5, D6: D_TVS, Diode_SMD:D_0603_1608Metric_Pad1.05x0.95mm_HandSolder, symbol Device:D_TVS
Connections:
- net GND: now also D5.1 (A1), D6.1 (A1)
- net POT1: now also D5.2 (A2)
- net POT2: now also D6.2 (A2)
Changed lines of the file:
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@@
   (junction (at 80.01 53.34) (diameter 0) (color 0 0 0 0)
   )
+  (junction (at 90.17 115.57) (diameter 0) (color 0 0 0 0)
+  )
   (junction (at 116.84 55.88) (diameter 0) (color 0 0 0 0)
   )
@@
   (junction (at 130.81 118.11) (diameter 0) (color 0 0 0 0)
   )
-  (junction (at 86.36 115.57) (diameter 0) (color 0 0 0 0)
-  )
   (junction (at 129.54 55.88) (diameter 0) (color 0 0 0 0)
   )
-  (junction (at 86.36 53.34) (diameter 0) (color 0 0 0 0)
+  (junction (at 90.17 53.34) (diameter 0) (color 0 0 0 0)
   )
   (wire (pts (xy 130.81 118.11) (xy 134.62 118.11))
@@
     (stroke (width 0) (type default) (color 0 0 0 0))
   )
+  (wire (pts (xy 90.17 123.19) (xy 90.17 130.302))
+    (stroke (width 0) (type default) (color 0 0 0 0))
+  )
   (wire (pts (xy 118.11 118.11) (xy 119.38 118.11))
     (stroke (width 0) (type default) (color 0 0 0 0))
@@
     (stroke (width 0) (type default) (color 0 0 0 0))
   )
-  (wire (pts (xy 101.6 115.57) (xy 86.36 115.57))
+  (wire (pts (xy 80.01 115.57) (xy 90.17 115.57))
     (stroke (width 0) (type default) (color 0 0 0 0))
   )
@@
     (stroke (width 0) (type default) (color 0 0 0 0))
   )
+  (wire (pts (xy 90.17 60.96) (xy 90.17 62.23))
+    (stroke (width 0) (type default) (color 0 0 0 0))
+  )
   (wire (pts (xy 130.81 125.73) (xy 130.81 128.27))
     (stroke (width 0) (type default) (color 0 0 0 0))
@@
     (stroke (width 0) (type default) (color 0 0 0 0))
   )
-  (wire (pts (xy 90.17 124.46) (xy 90.17 131.445))
-    (stroke (width 0) (type default) (color 0 0 0 0))
-  )
   (wire (pts (xy 118.11 118.11) (xy 118.11 134.62))
     (stroke (width 0) (type default) (color 0 0 0 0))
@@
     (stroke (width 0) (type default) (color 0 0 0 0))
   )
-  (wire (pts (xy 100.33 53.34) (xy 86.36 53.34))
-    (stroke (width 0) (type default) (color 0 0 0 0))
-  )
-  (wire (pts (xy 86.36 53.34) (xy 80.01 53.34))
+  (wire (pts (xy 80.01 53.34) (xy 90.17 53.34))
+    (stroke (width 0) (type default) (color 0 0 0 0))
+  )
+  (wire (pts (xy 90.17 115.57) (xy 101.6 115.57))
     (stroke (width 0) (type default) (color 0 0 0 0))
   )
@@
     (stroke (width 0) (type default) (color 0 0 0 0))
   )
+  (wire (pts (xy 90.17 53.34) (xy 100.33 53.34))
+    (stroke (width 0) (type default) (color 0 0 0 0))
+  )
   (wire (pts (xy 125.73 55.88) (xy 129.54 55.88))
-    (stroke (width 0) (type default) (color 0 0 0 0))
-  )
-  (wire (pts (xy 86.36 115.57) (xy 80.01 115.57))
     (stroke (width 0) (type default) (color 0 0 0 0))
   )
@@
     (effects (font (size 1.27 1.27)) (justify right))
   )
-  (hierarchical_label "3V3_POT2" (shape input) (at 90.17 106.68 90)
-    (effects (font (size 1.27 1.27)) (justify left))
-  )
   (hierarchical_label "POT1" (shape input) (at 69.85 53.34 180)
     (effects (font (size 1.27 1.27)) (justify right))
   )
   (hierarchical_label "SENSOR1" (shape output) (at 133.35 55.88 0)
-    (effects (font (size 1.27 1.27)) (justify left))
-  )
-  (hierarchical_label "3V3_POT1" (shape input) (at 90.17 44.45 90)
     (effects (font (size 1.27 1.27)) (justify left))
   )
@@
     (pin "1")
   )
-  (symbol (lib_id "power:GND") (at 90.17 131.445 0) (unit 1)
-    (in_bom yes) (on_board yes)
-    (property "Reference" "#PWR029" (id 0) (at 90.17 137.795 0)
-      (effects (font (size 1.27 1.27)) hide)
-    )
-    (property "Value" "GND" (id 1) (at 90.297 135.8392 0))
-    (property "Footprint" "" (id 2) (at 90.17 131.445 0)
-      (effects (font (size 1.27 1.27)) hide)
-    )
-    (property "Datasheet" "" (id 3) (at 90.17 131.445 0)
+  (symbol (lib_id "power:GND") (at 90.17 130.302 0) (unit 1)
+    (in_bom yes) (on_board yes)
+    (property "Reference" "#PWR029" (id 0) (at 90.17 136.652 0)
+      (effects (font (size 1.27 1.27)) hide)
+    )
+    (property "Value" "GND" (id 1) (at 90.297 134.6962 0))
+    (property "Footprint" "" (id 2) (at 90.17 130.302 0)
+      (effects (font (size 1.27 1.27)) hide)
+    )
+    (property "Datasheet" "" (id 3) (at 90.17 130.302 0)
       (effects (font (size 1.27 1.27)) hide)
     )
@@
     (pin "2")
   )
-  (symbol (lib_id "Device:D_TVS_x2_AAC") (at 90.17 115.57 270) (unit 1)
-    (in_bom yes) (on_board yes)
-    (property "Reference" "D12" (id 0) (at 92.71 106.68 90)
-      (effects (font (size 1.27 1.27)) (justify left))
-    )
-    (property "Value" "D_TVS_x2_AAC" (id 1) (at 91.44 109.22 90)
-      (effects (font (size 1.27 1.27)) (justify left))
-    )
-    (property "Footprint" "Package_TO_SOT_SMD:SOT-23" (id 2) (at 90.17 111.76 0)
-      (effects (font (size 1.27 1.27)) hide)
-    )
-    (property "Datasheet" "~" (id 3) (at 90.17 111.76 0)
-      (effects (font (size 1.27 1.27)) hide)
-    )
-    (pin "1")
-    (pin "2")
-    (pin "3")
-  )
-  (symbol (lib_id "Device:D_TVS_x2_AAC") (at 90.17 53.34 270) (unit 1)
-    (in_bom yes) (on_board yes)
-    (property "Reference" "D11" (id 0) (at 91.44 43.18 90)
-      (effects (font (size 1.27 1.27)) (justify left))
-    )
-    (property "Value" "D_TVS_x2_AAC" (id 1) (at 90.17 45.72 90)
-      (effects (font (size 1.27 1.27)) (justify left))
-    )
-    (property "Footprint" "Package_TO_SOT_SMD:SOT-23" (id 2) (at 90.17 49.53 0)
-      (effects (font (size 1.27 1.27)) hide)
-    )
-    (property "Datasheet" "~" (id 3) (at 90.17 49.53 0)
-      (effects (font (size 1.27 1.27)) hide)
-    )
-    (pin "1")
-    (pin "2")
-    (pin "3")
-  )
   (symbol (lib_id "Device:R_Small") (at 80.01 55.88 0) (unit 1)
     (in_bom yes) (on_board yes)
@@
     (pin "1")
   )
+  (symbol (lib_id "Device:D_TVS") (at 90.17 119.38 90) (unit 1)
+    (in_bom yes) (on_board yes) (fields_autoplaced)
+    (property "Reference" "D6" (id 0) (at 92.71 118.1099 90)
+      (effects (font (size 1.27 1.27)) (justify right))
+    )
+    (property "Value" "D_TVS" (id 1) (at 92.71 120.6499 90)
+      (effects (font (size 1.27 1.27)) (justify right))
+    )
+    (property "Footprint" "Diode_SMD:D_0603_1608Metric_Pad1.05x0.95mm_HandSolder" (id 2) (at 90.17 119.38 0)
+      (effects (font (size 1.27 1.27)) hide)
+    )
+    (property "Datasheet" "~" (id 3) (at 90.17 119.38 0)
+      (effects (font (size 1.27 1.27)) hide)
+    )
+    (pin "1")
+    (pin "2")
+  )
+  (symbol (lib_id "Device:D_TVS") (at 90.17 57.15 90) (unit 1)
+    (in_bom yes) (on_board yes) (fields_autoplaced)
+    (property "Reference" "D5" (id 0) (at 92.71 55.8799 90)
+      (effects (font (size 1.27 1.27)) (justify right))
+    )
+    (property "Value" "D_TVS" (id 1) (at 92.71 58.4199 90)
+      (effects (font (size 1.27 1.27)) (justify right))
+    )
+    (property "Footprint" "Diode_SMD:D_0603_1608Metric_Pad1.05x0.95mm_HandSolder" (id 2) (at 90.17 57.15 0)
+      (effects (font (size 1.27 1.27)) hide)
+    )
+    (property "Datasheet" "~" (id 3) (at 90.17 57.15 0)
+      (effects (font (size 1.27 1.27)) hide)
+    )
+    (pin "1")
+    (pin "2")
+  )
 )
