File: Hardware/Connectros.kicad_sch (KiCad schematic)
At the start: 7 parts, among them J4 Sygnały, J5 Diagnostyka, J8 Zasilanie+CAN

Commit message: PCB layout and routing
Connections:
- net +24V: now also J8.5 (Pin_5); no longer J8.1 (Pin_1)
Other:
- note added: "+24F1"
- note removed: "+24F3"
Changed lines of the file:
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@@
   (no_connect (at 79.375 78.105))
   (no_connect (at 224.79 80.01))
-  (no_connect (at 237.49 85.09))
   (no_connect (at 237.49 82.55))
   (no_connect (at 237.49 100.33))
@@
   (no_connect (at 79.375 85.725))
   (no_connect (at 114.3 95.885))
+  (no_connect (at 237.49 80.01))
   (no_connect (at 114.3 98.425))
   (no_connect (at 79.375 83.185))
@@
     (stroke (width 0) (type default) (color 0 0 0 0))
   )
+  (wire (pts (xy 237.49 85.09) (xy 265.43 85.09))
+    (stroke (width 0) (type default) (color 0 0 0 0))
+  )
   (polyline (pts (xy 105.41 85.725) (xy 107.95 85.725))
     (stroke (width 0) (type default) (color 0 0 0 0))
@@
     (stroke (width 0) (type default) (color 0 0 0 0))
   )
-  (wire (pts (xy 237.49 80.01) (xy 259.715 80.01))
-    (stroke (width 0) (type default) (color 0 0 0 0))
-  )
   (wire (pts (xy 186.055 92.71) (xy 191.77 92.71))
     (stroke (width 0) (type default) (color 0 0 0 0))
@@
     (effects (font (size 1.27 1.27)) (justify left bottom))
   )
+  (text "+24F1" (at 239.522 80.518 0)
+    (effects (font (size 1.27 1.27)) (justify left bottom))
+  )
   (text "PITOT2" (at 65.405 70.485 180)
     (effects (font (size 1.27 1.27)) (justify right bottom))
@@
   (text "INERTIA\n" (at 65.405 106.045 180)
     (effects (font (size 1.27 1.27)) (justify right bottom))
-  )
-  (text "+24F3\n" (at 239.395 85.09 0)
-    (effects (font (size 1.27 1.27)) (justify left bottom))
   )
   (text "S21" (at 80.645 93.345 0)
@@
     (pin "1")
     (pin "2")
+  )
+  (symbol (lib_id "power:+24V") (at 265.43 85.09 270) (unit 1)
+    (in_bom yes) (on_board yes) (fields_autoplaced)
+    (property "Reference" "#PWR0111" (id 0) (at 261.62 85.09 0)
+      (effects (font (size 1.27 1.27)) hide)
+    )
+    (property "Value" "+24V" (id 1) (at 268.605 85.0899 90)
+      (effects (font (size 1.27 1.27)) (justify left))
+    )
+    (property "Footprint" "" (id 2) (at 265.43 85.09 0)
+      (effects (font (size 1.27 1.27)) hide)
+    )
+    (property "Datasheet" "" (id 3) (at 265.43 85.09 0)
+      (effects (font (size 1.27 1.27)) hide)
+    )
+    (pin "1")
   )
   (symbol (lib_id "power:GND") (at 273.05 92.71 90) (unit 1)
@@
     (pin "9")
   )
-  (symbol (lib_id "power:+24V") (at 259.715 80.01 270) (unit 1)
-    (in_bom yes) (on_board yes) (fields_autoplaced)
-    (property "Reference" "#PWR0111" (id 0) (at 255.905 80.01 0)
-      (effects (font (size 1.27 1.27)) hide)
-    )
-    (property "Value" "+24V" (id 1) (at 262.89 80.0099 90)
-      (effects (font (size 1.27 1.27)) (justify left))
-    )
-    (property "Footprint" "" (id 2) (at 259.715 80.01 0)
-      (effects (font (size 1.27 1.27)) hide)
-    )
-    (property "Datasheet" "" (id 3) (at 259.715 80.01 0)
-      (effects (font (size 1.27 1.27)) hide)
-    )
-    (pin "1")
-  )
   (symbol (lib_id "conn_02x20_odd_even:Conn_02x20_Odd_Even") (at 71.755 90.805 0) (unit 1)

Commit message: Deleted 24V section
Parts:
- R13: value 220R -> 0R
- R17: value 0R -> 220R
Connections:
- net +5V: now reaches J8.2 (Pin_2)
- no-connect marks 62 -> 61
Changed lines of the file:
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@@
   (no_connect (at 66.675 83.185))
   (no_connect (at 79.375 78.105))
-  (no_connect (at 224.79 80.01))
   (no_connect (at 237.49 82.55))
   (no_connect (at 237.49 100.33))
@@
     (stroke (width 0) (type default) (color 0 0 0 0))
   )
+  (wire (pts (xy 224.79 80.01) (xy 203.962 80.01))
+    (stroke (width 0) (type default) (color 0 0 0 0))
+  )
   (wire (pts (xy 220.98 102.87) (xy 218.44 102.87))
     (stroke (width 0) (type default) (color 0 0 0 0))
@@
     (effects (font (size 1.27 1.27)) (justify left bottom))
   )
-  (text "+5V" (at 223.52 80.01 180)
+  (text "+5V" (at 223.012 75.692 180)
     (effects (font (size 1.27 1.27)) (justify right bottom))
   )
@@
     )
   )
+  (symbol (lib_id "power:+5V") (at 203.962 80.01 90) (unit 1)
+    (in_bom yes) (on_board yes) (fields_autoplaced)
+    (property "Reference" "#PWR0113" (id 0) (at 207.772 80.01 0)
+      (effects (font (size 1.27 1.27)) hide)
+    )
+    (property "Value" "+5V" (id 1) (at 200.66 80.0099 90)
+      (effects (font (size 1.27 1.27)) (justify left))
+    )
+    (property "Footprint" "" (id 2) (at 203.962 80.01 0)
+      (effects (font (size 1.27 1.27)) hide)
+    )
+    (property "Datasheet" "" (id 3) (at 203.962 80.01 0)
+      (effects (font (size 1.27 1.27)) hide)
+    )
+    (pin "1")
+  )
   (symbol (lib_id "Device:R") (at 262.255 92.71 270) (unit 1)
     (in_bom yes) (on_board yes)
     (property "Reference" "R17" (id 0) (at 260.985 95.25 90))
-    (property "Value" "0R" (id 1) (at 260.985 97.155 90))
+    (property "Value" "220R" (id 1) (at 260.985 97.155 90))
     (property "Footprint" "Resistor_SMD:R_1206_3216Metric" (id 2) (at 262.255 90.932 90)
       (effects (font (size 1.27 1.27)) hide)
@@
     (in_bom yes) (on_board yes)
     (property "Reference" "R13" (id 0) (at 196.85 95.25 90))
-    (property "Value" "220R" (id 1) (at 195.58 97.155 90))
+    (property "Value" "0R" (id 1) (at 195.58 97.155 90))
     (property "Footprint" "Resistor_SMD:R_1206_3216Metric" (id 2) (at 195.58 94.488 90)
       (effects (font (size 1.27 1.27)) hide)

Commit message: Generated BOM
Parts:
- R11, R13, R15, R17: footprint Resistor_SMD:R_1206_3216Metric -> Resistor_SMD:R_0603_1608Metric_Pad0.98x0.95mm_HandSolder
Connections:
- net RST renamed NRST
Changed lines of the file:
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@@
     )
   )
-  (global_label "RST" (shape input) (at 133.35 85.725 0) (fields_autoplaced)
+  (global_label "NRST" (shape input) (at 133.35 85.725 0) (fields_autoplaced)
     (effects (font (size 1.27 1.27)) (justify left))
-    (property "Intersheet References" "${INTERSHEET_REFS}" (id 0) (at 139.1213 85.6456 0)
+    (property "Intersheet References" "${INTERSHEET_REFS}" (id 0) (at 140.4518 85.6456 0)
       (effects (font (size 1.27 1.27)) (justify left) hide)
     )
@@
     (property "Reference" "R17" (id 0) (at 260.985 95.25 90))
     (property "Value" "220R" (id 1) (at 260.985 97.155 90))
-    (property "Footprint" "Resistor_SMD:R_1206_3216Metric" (id 2) (at 262.255 90.932 90)
+    (property "Footprint" "Resistor_SMD:R_0603_1608Metric_Pad0.98x0.95mm_HandSolder" (id 2) (at 262.255 90.932 90)
       (effects (font (size 1.27 1.27)) hide)
     )
@@
     (property "Reference" "R11" (id 0) (at 196.85 88.265 90))
     (property "Value" "220R" (id 1) (at 195.58 86.36 90))
-    (property "Footprint" "Resistor_SMD:R_1206_3216Metric" (id 2) (at 195.58 91.948 90)
+    (property "Footprint" "Resistor_SMD:R_0603_1608Metric_Pad0.98x0.95mm_HandSolder" (id 2) (at 195.58 91.948 90)
       (effects (font (size 1.27 1.27)) hide)
     )
@@
     (property "Reference" "R15" (id 0) (at 260.985 88.265 90))
     (property "Value" "0R" (id 1) (at 260.985 86.36 90))
-    (property "Footprint" "Resistor_SMD:R_1206_3216Metric" (id 2) (at 262.255 88.392 90)
+    (property "Footprint" "Resistor_SMD:R_0603_1608Metric_Pad0.98x0.95mm_HandSolder" (id 2) (at 262.255 88.392 90)
       (effects (font (size 1.27 1.27)) hide)
     )
@@
     (property "Reference" "R13" (id 0) (at 196.85 95.25 90))
     (property "Value" "0R" (id 1) (at 195.58 97.155 90))
-    (property "Footprint" "Resistor_SMD:R_1206_3216Metric" (id 2) (at 195.58 94.488 90)
-      (effects (font (size 1.27 1.27)) hide)
-    )
+    (property "Footprint" "Resistor_SMD:R_0603_1608Metric_Pad0.98x0.95mm_HandSolder" (id 2) (at 195.58 94.488 90)
+      (effects (font (size 1.27 1.27)) hide)
+    )
